File: MPPT_V3.kicad_sch (KiCad schematic)
At the start: 43 parts, among them CN1 XT60PW-M, CN2 XT60PW-M, U15 TP181A1-CR, U24 LM2901, U8 TP181A1-CR

Commit message: latest version with PWM fan and thermistors for each FET bank
Parts:
- C10, C11, C40, C41, C42, C43, C45, C46: LCSC Part (none) -> C880603
- C47, C49, C51, C52, C53, C54, C55, C56, C57, C58, C62, C63: LCSC Part (none) -> C5156756
- C59, C60, C66, C67: now left out of the parts list
- R20, R28: LCSC Part (none) -> C500733
- R24, R26: LCSC Part (none) -> C103915
- R25, R27, R41, R42, R43, R44: LCSC Part (none) -> C2930007
- U24: footprint (none) -> easyeda2kicad:SOP-14_L8.6-W3.9-P1.27-LS6.0-BL-1; LCSC Part (none) -> C5145307
- U24: LCSC Part (none) -> C5145307

Commit message: production version v3
Other:
- sheet fet_drivers_B ports: added none; removed Charge_pump_IN
Changed lines of the file:
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@@
 	(wire
 		(pts
-			(xy 181.61 44.45) (xy 176.53 44.45)
-		)
-		(stroke
-			(width 0)
-			(type default)
-		)
-	)
-	(wire
-		(pts
 			(xy 111.76 189.23) (xy 111.76 191.77)
 		)
@@
 	(wire
 		(pts
-			(xy 144.78 83.82) (xy 140.97 83.82)
-		)
-		(stroke
-			(width 0)
-			(type default)
-		)
-	)
-	(wire
-		(pts
 			(xy 154.94 191.77) (xy 154.94 196.85)
 		)
@@
 	(wire
 		(pts
-			(xy 140.97 83.82) (xy 140.97 59.69)
-		)
-		(stroke
-			(width 0)
-			(type default)
-		)
-	)
-	(wire
-		(pts
 			(xy 325.12 163.83) (xy 334.01 163.83)
 		)
@@
 	(wire
 		(pts
-			(xy 140.97 59.69) (xy 181.61 59.69)
-		)
-		(stroke
-			(width 0)
-			(type default)
-		)
-	)
-	(wire
-		(pts
 			(xy 82.55 185.42) (xy 87.63 185.42)
 		)
@@
 	(wire
 		(pts
-			(xy 181.61 59.69) (xy 181.61 44.45)
-		)
-		(stroke
-			(width 0)
-			(type default)
-		)
-	)
-	(wire
-		(pts
 			(xy 111.76 135.89) (xy 120.65 135.89)
 		)
@@
 			)
 		)
-		(pin "Charge_pump_IN" input
-			(at 144.78 83.82 180)
-			(effects
-				(font
-					(size 1.27 1.27)
-				)
-				(justify left)
-			)
-		)
